Commit message: Receive sensor media, plot in rviz

File: urdf/robot.urdf (robot description, URDF)
Before this commit: robot robot, 6 links, 5 joints
Links:
- added link range0; collision box size=0.01 0.03 0.01; visual box size=0.01 0.03 0.01
- added link range10; collision box size=0.01 0.03 0.01; visual box size=0.01 0.03 0.01
- added link range11; collision box size=0.01 0.03 0.01; visual box size=0.01 0.03 0.01
- added link range2; collision box size=0.01 0.03 0.01; visual box size=0.01 0.03 0.01
- added link range3; collision box size=0.01 0.03 0.01; visual box size=0.01 0.03 0.01
- added link range4; collision box size=0.01 0.03 0.01; visual box size=0.01 0.03 0.01
- added link range5; collision box size=0.01 0.03 0.01; visual box size=0.01 0.03 0.01
- added link range6; collision box size=0.01 0.03 0.01; visual box size=0.01 0.03 0.01
- added link range7; collision box size=0.01 0.03 0.01; visual box size=0.01 0.03 0.01
- added link range8; collision box size=0.01 0.03 0.01; visual box size=0.01 0.03 0.01
- added link range9; collision box size=0.01 0.03 0.01; visual box size=0.01 0.03 0.01
Joints:
- added joint top_to_range0: type fixed, parent top, child range0, origin xyz=0.05 0 .02 rpy=0 0 0, limit effort=100 velocity=100
- added joint top_to_range10: type fixed, parent top, child range10, origin xyz=0.025 0.0433012701892219 .02 rpy=0 0 -5.235987756, limit effort=100 velocity=100
- added joint top_to_range11: type fixed, parent top, child range11, origin xyz=0.0433012701892219 0.025 -.02 rpy=0 0 -5.7595865316, limit effort=100 velocity=100
- added joint top_to_range2: type fixed, parent top, child range2, origin xyz=0.025 -0.0433012701892219 .02 rpy=0 0 -1.0471975512, limit effort=100 velocity=100
- added joint top_to_range3: type fixed, parent top, child range3, origin xyz=3.06161699786838E-018 -0.05 -.02 rpy=0 0 -1.5707963268, limit effort=100 velocity=100
- added joint top_to_range4: type fixed, parent top, child range4, origin xyz=-0.025 -0.0433012701892219 .02 rpy=0 0 -2.0943951024, limit effort=100 velocity=100
- added joint top_to_range5: type fixed, parent top, child range5, origin xyz=-0.0433012701892219 -0.025 -.02 rpy=0 0 -2.617993878, limit effort=100 velocity=100
- added joint top_to_range6: type fixed, parent top, child range6, origin xyz=-0.05 -6.12323399573677E-018 .02 rpy=0 0 -3.1415926536, limit effort=100 velocity=100
- added joint top_to_range7: type fixed, parent top, child range7, origin xyz=-0.0433012701892219 0.025 -.02 rpy=0 0 -3.6651914292, limit effort=100 velocity=100
- added joint top_to_range8: type fixed, parent top, child range8, origin xyz=-0.025 0.0433012701892219 .02 rpy=0 0 -4.1887902048, limit effort=100 velocity=100
- added joint top_to_range9: type fixed, parent top, child range9, origin xyz=-9.18485099360515E-018 0.05 -.02 rpy=0 0 -4.7123889804, limit effort=100 velocity=100
- joint top_to_range1: origin xyz=0.05 0 .02 rpy=0 0 0 -> xyz=0.0433012701892219 -0.025 -.02 rpy=0 0 -0.5235987756
