File: board/v3/mctrli2c.brd (EAGLE design)
At the start: 33.7 x 43.9 mm, 15 parts, among them IC1 L293DD, U1 ATTINY861-20SU

Commit message: Updates to the board and cad
Routing:
- net M1_T1: track 0.00 -> 17.1 mm, vias 0 -> 1
- net M2_T1: track 0.00 -> 15.3 mm, vias 0 -> 1
- net M1_T2: track 0.00 -> 8.52 mm, vias 0 -> 1
- net M2_T2: track 0.00 -> 8.32 mm, vias 0 -> 1
- net GND: track 22.0 -> 22.1 mm, vias 11 -> 14
Other:
- board text added: "L293DD"
- board text added: "attiny861A"
